File: pcb/grbl_controller.kicad_sch (KiCad schematic)
At the start: 40 parts, among them J1 DA15_Plug_MountingHoles, U1 firebeetle_esp32, U2 EL817, U3 EL817, U4 EL817, U5 EL817, U6 74LS07, U7 74LS07

Commit message: Finished PCB layout.
Parts:
- C1, C2, C3, C4, C5, C6: footprint (none) -> Capacitor_SMD:C_0805_2012Metric
- J1: footprint (none) -> Connector_Dsub:DSUB-15_Male_Horizontal_P2.77x2.84mm_EdgePinOffset9.90mm_Housed_MountingHolesOffset11.32mm; MPN (none) -> L717SDA15P1ACH4R; OC_MOUSER (none) -> 523-L717SDA15P1ACH4R
- R1, R10, R11, R12, R13, R14, R15, R16, R17, R2, R3, R4, R5, R6, R7, R8, R9: footprint (none) -> Resistor_SMD:R_0805_2012Metric
- U6, U7: footprint (none) -> Package_SO:SOIC-14_3.9x8.7mm_P1.27mm
Connections:
- net +5V: now also U1.18 (VCC)
- net GND: now also J1.0 (PAD), U1.15 (GND)
- net at U6.8: now also R14.1; no longer R12.1
- net G_Y_PULSE: now reaches U6.9
- net G_Y_PULSE: now also U1.9 (IO5/D8)
- net G_Y_LIMIT: now reaches R5.2, U4.4
- net G_Y_LIMIT: now also U1.24 (BCLK/IO14)
- net at U6.12: now also R10.1; no longer R14.1
- net G_Y_DIR: now reaches U7.5
- net G_Y_DIR: now also U1.20 (LRCK/IO17)
- net at U7.6: now also R15.1; no longer R17.1
- net G_Z_LIMIT: now reaches R2.2, U2.4
- net G_Z_LIMIT: now also U1.23 (MCLK/IO12)
- net G_SPINDLE_M: now reaches U6.1
- net G_SPINDLE_M: now also U1.4 (IO26/D3)
- net G_TOOL_SENSE: now reaches R3.2, U3.4
- net G_TOOL_SENSE: now also U1.26 (SDA/IO21)
- net G_X_DIR: now reaches U7.1
- net G_X_DIR: now also U1.22 (DO/IO4)
- net at U7.2: now also R17.1; no longer R15.1
- net G_X_LIMIT: now reaches R7.2, U5.4
- net G_X_LIMIT: now also U1.25 (SCL/IO22)
- net G_Z_DIR: now reaches U6.5
- net G_Z_DIR: now also U1.10 (IO2/D9)
- net at U6.6: now also R13.1; no longer R11.1
- net G_Z_PULSE: now reaches U1.21 (D1/IO16)
- net G_Z_PULSE: now also U7.3
- net G_SPINDLE_H: now reaches U1.3 (IO25/D2)
- net G_SPINDLE_H: now also U6.13
- net G_SPINDLE_L: now reaches U1.5 (IO27/D4)
- net G_SPINDLE_L: now also U6.3
- net G_X_PULSE: now reaches U1.8 (IO13/D7)
- net G_X_PULSE: now also U6.11
- net at U6.4: now also R11.1; no longer R10.1
- net at U6.10: now also R12.1; no longer R13.1
- no-connect marks 0 -> 18
Other:
- note added: "SPI FLASH PIN"
- moved on the sheet: D1, D3, D4, D5, D6, R11, R12, R13, R14, R9, U6A, U6B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
